File: Schematics/NuceloBoard/ESP_Schematics.kicad_sch (KiCad schematic)
At the start: 5 parts, among them J1 Conn_01x04_Male, J2 Conn_01x04_Male

Commit message: added NuceloBoard Schematics
Other:
- note added: "Battery Monitor"
Changed lines of the file:
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@@
+    (stroke (width 0) (type default) (color 0 0 0 0))
+  )
+  (wire (pts (xy 176.53 66.04) (xy 187.96 66.04))
     (stroke (width 0) (type default) (color 0 0 0 0))
   )
@@
     (effects (font (size 1.27 1.27)) (justify left bottom))
   )
+  (text "Battery Monitor" (at 179.07 64.77 0)
+    (effects (font (size 1.27 1.27)) (justify left bottom))
+  )
