File: Schematics/ESP/Peripherals.kicad_sch (KiCad schematic)
At the start: 38 parts, among them J3 Screw_Terminal_01x02, J4 Conn_01x02_Male, J5 Conn_01x02_Male, J6 Screw_Terminal_01x02 Fan, J8 Screw_Terminal_01x04, Q17 IRF540N, Q3 AO3401A, U4 DRV8871DDA, U5 LM2596S-5, U6 DRV8871DDA

Commit message: fixed BOM
Parts:
- C11: footprint Capacitor_Tantalum_SMD:CP_EIA-7343-31_Kemet-D_Pad2.25x2.55mm_HandSolder -> Capacitor_SMD:C_0603_1608Metric_Pad1.08x0.95mm_HandSolder
- C12, C13, C8, C9: footprint Capacitor_THT:CP_Radial_D10.0mm_P5.00mm -> Capacitor_SMD:C_1206_3216Metric_Pad1.33x1.80mm_HandSolder
- C7: footprint Capacitor_Tantalum_SMD:CP_EIA-7343-31_Kemet-D_Pad2.25x2.55mm_HandSolder -> Capacitor_SMD:C_1206_3216Metric_Pad1.33x1.80mm_HandSolder
Connections:
- net Battery+: now also F1.2, U4.5 (VM); no longer C11.1, C12.1
- net at F1.2, U6.5 (VM): now also C11.1, C12.1
Other:
- moved on the sheet: F1
Changed lines of the file:
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@@
   (junction (at 93.98 123.19) (diameter 0) (color 0 0 0 0)
   )
+  (junction (at 43.18 152.4) (diameter 0) (color 0 0 0 0)
+  )
   (junction (at 155.575 54.61) (diameter 0) (color 0 0 0 0)
   )
@@
     (stroke (width 0) (type default))
   )
+  (wire (pts (xy 43.18 152.4) (xy 45.72 152.4))
+    (stroke (width 0) (type default))
+  )
   (wire (pts (xy 157.48 64.77) (xy 157.48 66.04))
     (stroke (width 0) (type default))
@@
     (stroke (width 0) (type default))
   )
+  (wire (pts (xy 55.88 152.4) (xy 71.12 152.4))
+    (stroke (width 0) (type default))
+  )
   (wire (pts (xy 157.48 71.12) (xy 157.48 73.66))
     (stroke (width 0) (type default))
@@
     (stroke (width 0) (type default))
   )
-  (wire (pts (xy 85.09 123.19) (xy 93.98 123.19))
-    (stroke (width 0) (type default))
-  )
   (wire (pts (xy 50.8 160.02) (xy 50.8 162.56))
     (stroke (width 0) (type default))
@@
     (stroke (width 0) (type default))
   )
-  (wire (pts (xy 119.38 123.19) (xy 128.27 123.19))
-    (stroke (width 0) (type default))
-  )
   (wire (pts (xy 247.65 132.715) (xy 247.65 130.81))
     (stroke (width 0) (type default))
@@
     (stroke (width 0) (type default))
   )
+  (wire (pts (xy 92.71 123.19) (xy 93.98 123.19))
+    (stroke (width 0) (type default))
+  )
   (wire (pts (xy 52.07 170.18) (xy 68.58 170.18))
     (stroke (width 0) (type default))
@@
     (stroke (width 0) (type default))
   )
+  (wire (pts (xy 104.14 123.19) (xy 128.27 123.19))
+    (stroke (width 0) (type default))
+  )
   (wire (pts (xy 157.48 64.77) (xy 148.59 64.77))
     (stroke (width 0) (type default))
@@
     (stroke (width 0) (type default))
   )
-  (wire (pts (xy 104.14 123.19) (xy 111.76 123.19))
-    (stroke (width 0) (type default))
-  )
   (wire (pts (xy 240.03 154.94) (xy 240.03 153.035))
     (stroke (width 0) (type default))
@@
     (stroke (width 0) (type default))
   )
-  (wire (pts (xy 35.56 152.4) (xy 45.72 152.4))
-    (stroke (width 0) (type default))
-  )
   (wire (pts (xy 86.36 54.61) (xy 86.36 64.77))
     (stroke (width 0) (type default))
@@
     (stroke (width 0) (type default))
   )
-  (wire (pts (xy 55.88 152.4) (xy 60.96 152.4))
+  (wire (pts (xy 55.88 152.4) (xy 45.72 152.4))
     (stroke (width 0) (type default))
   )
@@
     (stroke (width 0) (type default))
   )
+  (wire (pts (xy 35.56 152.4) (xy 43.18 152.4))
+    (stroke (width 0) (type default))
+  )
   (wire (pts (xy 78.74 49.53) (xy 83.185 49.53))
     (stroke (width 0) (type default))
@@
     (stroke (width 0) (type default))
   )
-  (wire (pts (xy 68.58 152.4) (xy 71.12 152.4))
-    (stroke (width 0) (type default))
-  )
   (wire (pts (xy 210.82 58.42) (xy 210.82 68.58))
     (stroke (width 0) (type default))
@@
   )
   (wire (pts (xy 240.03 150.495) (xy 253.365 150.495))
-    (stroke (width 0) (type default))
-  )
-  (wire (pts (xy 55.88 152.4) (xy 45.72 152.4))
     (stroke (width 0) (type default))
   )
@@
     )
   )
-  (symbol (lib_id "Device:Polyfuse") (at 64.77 152.4 90) (unit 1)
-    (in_bom yes) (on_board yes) (dnp no) (fields_autoplaced)
-    (property "Reference" "F1" (at 64.77 147.32 90)
-      (effects (font (size 1.27 1.27)))
-    )
-    (property "Value" "1.6A" (at 64.77 149.86 90)
-      (effects (font (size 1.27 1.27)))
-    )
-    (property "Footprint" "Fuse:Fuse_1812_4532Metric_Pad1.30x3.40mm_HandSolder" (at 69.85 151.13 0)
+  (symbol (lib_id "Device:Polyfuse") (at 39.37 152.4 90) (unit 1)
+    (in_bom yes) (on_board yes) (dnp no) (fields_autoplaced)
+    (property "Reference" "F1" (at 39.37 147.32 90)
+      (effects (font (size 1.27 1.27)))
+    )
+    (property "Value" "1.6A" (at 39.37 149.86 90)
+      (effects (font (size 1.27 1.27)))
+    )
+    (property "Footprint" "Fuse:Fuse_1812_4532Metric_Pad1.30x3.40mm_HandSolder" (at 44.45 151.13 0)
       (effects (font (size 1.27 1.27)) (justify left) hide)
     )
-    (property "Datasheet" "https://www.belfuse.com/resources/datasheets/circuitprotection/ds-cp-0zcg-series.pdf" (at 64.77 152.4 0)
-      (effects (font (size 1.27 1.27)) hide)
-    )
-    (property "digikey link" "https://www.digikey.fi/en/products/detail/bel-fuse-inc/0ZCG0150BF2C/4156109" (at 64.77 152.4 90)
-      (effects (font (size 1.27 1.27)) hide)
-    )
-    (property "Price" "0,86" (at 64.77 152.4 0)
+    (property "Datasheet" "https://www.belfuse.com/resources/datasheets/circuitprotection/ds-cp-0zcg-series.pdf" (at 39.37 152.4 0)
+      (effects (font (size 1.27 1.27)) hide)
+    )
+    (property "digikey link" "https://www.digikey.fi/en/products/detail/bel-fuse-inc/0ZCG0150BF2C/4156109" (at 39.37 152.4 90)
+      (effects (font (size 1.27 1.27)) hide)
+    )
+    (property "Price" "0,86" (at 39.37 152.4 0)
       (effects (font (size 1.27 1.27)) hide)
     )
@@
       (effects (font (size 1.27 1.27)) (justify left))
     )
-    (property "Footprint" "Capacitor_Tantalum_SMD:CP_EIA-7343-31_Kemet-D_Pad2.25x2.55mm_HandSolder" (at 45.72 157.48 0)
+    (property "Footprint" "Capacitor_SMD:C_1206_3216Metric_Pad1.33x1.80mm_HandSolder" (at 45.72 157.48 0)
       (effects (font (size 1.27 1.27)) hide)
     )
@@
     )
   )
-  (symbol (lib_id "Device:Polyfuse") (at 115.57 123.19 90) (unit 1)
-    (in_bom yes) (on_board yes) (dnp no) (fields_autoplaced)
-    (property "Reference" "F1" (at 115.57 118.11 90)
-      (effects (font (size 1.27 1.27)))
-    )
-    (property "Value" "1.6A" (at 115.57 120.65 90)
-      (effects (font (size 1.27 1.27)))
-    )
-    (property "Footprint" "Fuse:Fuse_1812_4532Metric_Pad1.30x3.40mm_HandSolder" (at 120.65 121.92 0)
+  (symbol (lib_id "Device:Polyfuse") (at 88.9 123.19 90) (unit 1)
+    (in_bom yes) (on_board yes) (dnp no) (fields_autoplaced)
+    (property "Reference" "F1" (at 88.9 118.11 90)
+      (effects (font (size 1.27 1.27)))
+    )
+    (property "Value" "1.6A" (at 88.9 120.65 90)
+      (effects (font (size 1.27 1.27)))
+    )
+    (property "Footprint" "Fuse:Fuse_1812_4532Metric_Pad1.30x3.40mm_HandSolder" (at 93.98 121.92 0)
       (effects (font (size 1.27 1.27)) (justify left) hide)
     )
-    (property "Datasheet" "https://www.belfuse.com/resources/datasheets/circuitprotection/ds-cp-0zcg-series.pdf" (at 115.57 123.19 0)
-      (effects (font (size 1.27 1.27)) hide)
-    )
-    (property "digikey link" "https://www.digikey.fi/en/products/detail/bel-fuse-inc/0ZCG0150BF2C/4156109" (at 115.57 123.19 90)
-      (effects (font (size 1.27 1.27)) hide)
-    )
-    (property "Price" "0,86" (at 115.57 123.19 0)
+    (property "Datasheet" "https://www.belfuse.com/resources/datasheets/circuitprotection/ds-cp-0zcg-series.pdf" (at 88.9 123.19 0)
+      (effects (font (size 1.27 1.27)) hide)
+    )
+    (property "digikey link" "https://www.digikey.fi/en/products/detail/bel-fuse-inc/0ZCG0150BF2C/4156109" (at 88.9 123.19 90)
+      (effects (font (size 1.27 1.27)) hide)
+    )
+    (property "Price" "0,86" (at 88.9 123.19 0)
       (effects (font (size 1.27 1.27)) hide)
     )
@@
       (effects (font (size 1.27 1.27)) (justify left))
     )
-    (property "Footprint" "Capacitor_THT:CP_Radial_D10.0mm_P5.00mm" (at 104.14 143.51 0)
+    (property "Footprint" "Capacitor_SMD:C_1206_3216Metric_Pad1.33x1.80mm_HandSolder" (at 104.14 143.51 0)
       (effects (font (size 1.27 1.27)) hide)
     )
@@
       (effects (font (size 1.27 1.27)) (justify left))
     )
-    (property "Footprint" "Capacitor_Tantalum_SMD:CP_EIA-7343-31_Kemet-D_Pad2.25x2.55mm_HandSolder" (at 93.98 128.27 0)
+    (property "Footprint" "Capacitor_SMD:C_0603_1608Metric_Pad1.08x0.95mm_HandSolder" (at 93.98 128.27 0)
       (effects (font (size 1.27 1.27)) hide)
     )
@@
       (effects (font (size 1.27 1.27)) (justify left))
     )
-    (property "Footprint" "Capacitor_THT:CP_Radial_D10.0mm_P5.00mm" (at 55.88 157.48 0)
+    (property "Footprint" "Capacitor_SMD:C_1206_3216Metric_Pad1.33x1.80mm_HandSolder" (at 55.88 157.48 0)
       (effects (font (size 1.27 1.27)) hide)
     )
@@
       (effects (font (size 1.27 1.27)) (justify left))
     )
-    (property "Footprint" "Capacitor_THT:CP_Radial_D10.0mm_P5.00mm" (at 104.14 128.27 0)
+    (property "Footprint" "Capacitor_SMD:C_1206_3216Metric_Pad1.33x1.80mm_HandSolder" (at 104.14 128.27 0)
       (effects (font (size 1.27 1.27)) hide)
     )
@@
       (effects (font (size 1.27 1.27)) (justify left))
     )
-    (property "Footprint" "Capacitor_THT:CP_Radial_D10.0mm_P5.00mm" (at 52.07 173.99 0)
-      (effects (font (size 1.27 1.27)) hide)
-    )
+    (property "Footprint" "Capacitor_SMD:C_1206_3216Metric_Pad1.33x1.80mm_HandSolder" (at 52.07 173.99 0)
+      (effects (font (size 1.27 1.27)) hide)
+    )

Commit message: some pcb changes
Parts:
- removed J3: Screw_Terminal_01x02, TerminalBlock_Phoenix:TerminalBlock_Phoenix_PT-1,5-2-5.0-H_1x02_P5.00mm_Horizontal, symbol Connector:Screw_Terminal_01x02
- removed J8: Screw_Terminal_01x04, TerminalBlock_Phoenix:TerminalBlock_Phoenix_MKDS-1,5-4-5.08_1x04_P5.08mm_Horizontal, symbol Connector:Screw_Terminal_01x04
- added J12: Conn_01x02_Pin, Connector_PinSocket_1.00mm:PinSocket_1x02_P1.00mm_Vertical, symbol Connector:Conn_01x02_Pin
- added J3: Conn_01x04_Pin, Connector_PinHeader_1.00mm:PinHeader_1x04_P1.00mm_Vertical, symbol Connector:Conn_01x04_Pin
- C11: footprint Capacitor_SMD:C_0603_1608Metric_Pad1.08x0.95mm_HandSolder -> Capacitor_SMD:C_1206_3216Metric_Pad1.33x1.80mm_HandSolder
- F1: footprint Fuse:Fuse_1812_4532Metric_Pad1.30x3.40mm_HandSolder -> Fuse:Fuse_1206_3216Metric_Pad1.42x1.75mm_HandSolder
- F1: footprint Fuse:Fuse_1812_4532Metric_Pad1.30x3.40mm_HandSolder -> Fuse:Fuse_0603_1608Metric_Pad1.05x0.95mm_HandSolder
Connections:
- net Battery+: now also J12.1 (Pin_1), J3.1 (Pin_1); no longer C7.1, C9.1, F1.2, U4.5 (VM)
- net Cell1+: now also J3.3 (Pin_3)
- net Cell2+: now also J3.2 (Pin_2)
- net GND: now also J12.2 (Pin_2), J3.4 (Pin_4)
- new net: C7.1, C9.1, F1.2, U4.5 (VM)
Other:
- moved on the sheet: F1

Commit message: Changed schematics and PCB for shield
Parts:
- J12: footprint Connector_PinSocket_1.00mm:PinSocket_1x02_P1.00mm_Vertical -> Connector_PinSocket_2.54mm:PinSocket_1x02_P2.54mm_Vertical
- J3: footprint Connector_PinHeader_1.00mm:PinHeader_1x04_P1.00mm_Vertical -> Connector_PinHeader_2.54mm:PinHeader_1x04_P2.54mm_Vertical
Changed lines of the file:
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@@
       (effects (font (size 1.27 1.27)))
     )
-    (property "Footprint" "Connector_PinHeader_1.00mm:PinHeader_1x04_P1.00mm_Vertical" (at 257.81 149.86 0)
+    (property "Footprint" "Connector_PinHeader_2.54mm:PinHeader_1x04_P2.54mm_Vertical" (at 257.81 149.86 0)
       (effects (font (size 1.27 1.27)) hide)
     )
@@
       (effects (font (size 1.27 1.27)))
     )
-    (property "Footprint" "Connector_PinSocket_1.00mm:PinSocket_1x02_P1.00mm_Vertical" (at 255.27 128.27 0)
-      (effects (font (size 1.27 1.27)) hide)
-    )
+    (property "Footprint" "Connector_PinSocket_2.54mm:PinSocket_1x02_P2.54mm_Vertical" (at 255.27 128.27 0)
+      (effects (font (size 1.27 1.27)) hide)
+    )
