File: Schematics/ESP/ESP.kicad_pcb (KiCad board)
At the start: 2 copper layers, 40 parts, among them J3 Screw_Terminal_01x02, J6 Screw_Terminal_01x02 Fan, J8 Screw_Terminal_01x04, Q15 AO3401A, Q17 IRF540N, Q5 IRLB8721PBF, Q6 IRLB8721PBF, SW2 SW_Push, U1 AP9101CK, U2 AP9101CK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

Commit message: some pcb changes
Parts:
- removed J8: Screw_Terminal_01x04, TerminalBlock_Phoenix:TerminalBlock_Phoenix_MKDS-1,5-4-5.08_1x04_P5.08mm_Horizontal
- added C10: 10n, Capacitor_SMD:C_1206_3216Metric_Pad1.33x1.80mm_HandSolder, F.Cu at (129.6, 128.8)
- added C4: 100nF, Capacitor_SMD:C_1206_3216Metric_Pad1.33x1.80mm_HandSolder, F.Cu at (53.9, 141.8)
- added C5: 10n, Capacitor_SMD:C_1206_3216Metric_Pad1.33x1.80mm_HandSolder, F.Cu at (67.5, 139.6)
- added C6: 47u, Capacitor_SMD:C_1206_3216Metric_Pad1.33x1.80mm_HandSolder, F.Cu at (53.9, 139.1)
- added C8: 100nF, Capacitor_SMD:C_1206_3216Metric_Pad1.33x1.80mm_HandSolder, F.Cu at (140.8, 132.1)
- added C9: 47u, Capacitor_SMD:C_1206_3216Metric_Pad1.33x1.80mm_HandSolder, F.Cu at (138.0, 132.1)
- added F2: 1.6A, Fuse:Fuse_0603_1608Metric_Pad1.05x0.95mm_HandSolder, F.Cu at (55.6, 134.4)
- added F3: 1.6A, Fuse:Fuse_0603_1608Metric_Pad1.05x0.95mm_HandSolder, F.Cu at (144.1, 130.5)
- added F4: 0.72A, Fuse:Fuse_1206_3216Metric_Pad1.42x1.75mm_HandSolder, F.Cu at (155.0, 77.9)
- added J1: Barrel_Jack, RAPC722X:SWITCHCRAFT_RAPC722X, F.Cu at (229.5, 64.5)
- added J10: Conn_01x03_Socket, Connector_PinHeader_1.00mm:PinHeader_1x03_P1.00mm_Vertical, F.Cu at (90.2, 104.6)
- added J11: Conn_01x02_Pin, Connector_PinSocket_1.00mm:PinSocket_1x02_P1.00mm_Vertical, F.Cu at (106.1, 101.9)
- added J12: Conn_01x02_Pin, Connector_PinSocket_1.00mm:PinSocket_1x02_P1.00mm_Vertical, F.Cu at (48.6, 105.1)
- added J13: Conn_01x02_Pin, Connector_PinSocket_1.00mm:PinSocket_1x02_P1.00mm_Vertical, F.Cu at (280.6, 138.5)
- added J2: Conn_01x04_Male, Connector_PinSocket_1.00mm:PinSocket_1x04_P1.00mm_Vertical, F.Cu at (71.9, 104.5)
- added J4: Conn_01x02_Male, Connector_PinHeader_1.27mm:PinHeader_1x02_P1.27mm_Horizontal, F.Cu at (143.2, 124.3)
- added J5: Conn_01x02_Male, Connector_PinHeader_1.27mm:PinHeader_1x02_P1.27mm_Horizontal, F.Cu at (53.0, 146.3)
- added J7: Conn_01x04_Male, Connector_PinSocket_1.00mm:PinSocket_1x04_P1.00mm_Vertical, F.Cu at (75.7, 117.9)
- added J9: Conn_01x03_Socket, Connector_PinHeader_1.00mm:PinHeader_1x03_P1.00mm_Vertical, F.Cu at (125.1, 103.5)
- added R1: 2k, Resistor_SMD:R_1206_3216Metric_Pad1.30x1.75mm_HandSolder, F.Cu at (76.7, 113.9)
- added R15: 2k, Resistor_SMD:R_1206_3216Metric_Pad1.30x1.75mm_HandSolder, F.Cu at (67.4, 145.3)
- added R16: 39k, Resistor_SMD:R_1206_3216Metric_Pad1.30x1.75mm_HandSolder, F.Cu at (64.3, 135.3)
- added R17: 3k3, Resistor_SMD:R_1206_3216Metric_Pad1.30x1.75mm_HandSolder, F.Cu at (124.6, 127.5)
- added R18: 2k, Resistor_SMD:R_1206_3216Metric_Pad1.30x1.75mm_HandSolder, F.Cu at (128.6, 124.2)
- added R19: 39k, Resistor_SMD:R_1206_3216Metric_Pad1.30x1.75mm_HandSolder, F.Cu at (132.5, 132.3)
- added R20: 3k3, Resistor_SMD:R_1206_3216Metric_Pad1.30x1.75mm_HandSolder, F.Cu at (72.5, 141.2)
- C1, C2, C3: footprint Capacitor_Tantalum_SMD:CP_EIA-7343-31_Kemet-D_Pad2.25x2.55mm_HandSolder -> Capacitor_SMD:C_1206_3216Metric_Pad1.33x1.80mm_HandSolder
- J3: value Screw_Terminal_01x02 -> Conn_01x04_Pin; footprint TerminalBlock_Phoenix:TerminalBlock_Phoenix_PT-1,5-2-5.0-H_1x02_P5.00mm_Horizontal -> Connector_PinHeader_1.00mm:PinHeader_1x04_P1.00mm_Vertical
- R12, R13, R14: value 1k -> 10k
- moved U4 132.3 mm to (61.4, 142.3), turned to 180 degrees
- moved R7 129.9 mm to (71.3, 113.9)
- moved L1 116.1 mm to (191.2, 132.4), turned to 90 degrees
- moved R14 113.4 mm to (102.9, 79.0), turned to -90 degrees
- moved R12 109.5 mm to (105.9, 79.0), turned to 90 degrees
- moved R13 105.2 mm to (109.2, 79.0), turned to 90 degrees
- moved F1 104.6 mm to (238.1, 150.8), turned to 180 degrees
- moved Q15 102.9 mm to (210.2, 150.3), turned to 0 degrees
- moved D1 94.9 mm to (211.2, 141.3), turned to 180 degrees
- moved J3 90.2 mm to (280.0, 77.4)
- moved U5 87.5 mm to (212.7, 132.4), turned to 180 degrees
- moved U6 84.3 mm to (135.7, 125.5)
- moved Q5 70.9 mm to (246.2, 59.0)
- moved Q6 70.9 mm to (246.2, 64.9)
- moved SW2 70.9 mm to (264.8, 80.0)
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Connections:
- J3 pad 2: Battery- -> Cell2+
- Q17 pad 2: Net-(J6-Pin_2) -> Net-(Q17-D)
- U4 pad 5: Battery+ -> Net-(U4-VM)
- U6 pad 5: Battery+ -> Net-(U6-VM)
- U7 pad 36: unconnected-(U7-PC1-Pad36) -> Bumper Button 1
- U7 pad 72: unconnected-(U7-PC4-Pad72) -> Bumper Button 2
Other:
- board text added: "BLE"
- board text added: "Battery Charging circuit"
- board text added: "Battery Monitor"
- board text added: "Bumper 1"
- board text added: "Bumper 2"
- board text added: "FAN"
- board text added: "IR 1"
- board text added: "IR 2"
- board text added: "MPU"
- board text added: "Motor A"
- board text added: "Motor B"
- board text added: "Voltage Regulator"

Commit message: Can't Pull
Parts:
- moved Q5 45.6 mm to (243.3, 104.5), turned to 90 degrees
- moved SW2 39.3 mm to (228.7, 95.4), turned to -90 degrees
- moved U8 32.6 mm to (254.3, 104.2), turned to 180 degrees
- moved U3 31.0 mm to (263.1, 109.8), turned to 180 degrees
- moved R11 30.1 mm to (267.6, 86.0), turned to -90 degrees
- moved R5 28.9 mm to (268.0, 112.6), turned to -90 degrees
- moved R3 28.8 mm to (269.2, 77.3), turned to 180 degrees
- moved Q6 28.6 mm to (243.2, 93.4), turned to 90 degrees
- moved R6 25.1 mm to (269.3, 103.6)
- moved U1 24.8 mm to (262.8, 96.5), turned to 180 degrees
- moved R2 24.5 mm to (269.0, 91.2)
- moved R9 23.3 mm to (267.7, 99.1), turned to -90 degrees
- moved U9 22.7 mm to (254.2, 95.0), turned to 180 degrees
- moved C2 22.2 mm to (269.3, 81.3), turned to 180 degrees
- moved J1 21.0 mm to (247.2, 75.8), turned to -90 degrees
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
Commit message: Changed schematics and PCB for shield
Parts:
- removed U7: NUCLEO64-F411RE, Module:ST_Morpho_Connector_144_STLink
- added J14: Conn_02x19_Odd_Even, Connector_PinSocket_2.54mm:PinSocket_2x19_P2.54mm_Vertical, F.Cu at (82.3, 21.0)
- added J16: Conn_02x19_Odd_Even, Connector_PinSocket_2.54mm:PinSocket_2x19_P2.54mm_Vertical, F.Cu at (89.4, 21.0)
- added J2: Conn_01x06_Pin, Connector_PinSocket_2.54mm:PinSocket_1x06_P2.54mm_Vertical, F.Cu at (58.1, 65.9)
- added J7: Conn_01x07_Pin, Connector_PinSocket_2.54mm:PinSocket_1x07_P2.54mm_Vertical, F.Cu at (116.9, 46.1)
- J13: footprint Connector_PinSocket_1.00mm:PinSocket_1x02_P1.00mm_Vertical -> Connector_PinSocket_2.54mm:PinSocket_1x02_P2.54mm_Vertical
- J2, J7: footprint Connector_PinSocket_1.00mm:PinSocket_1x04_P1.00mm_Vertical -> Connector_PinSocket_2.54mm:PinSocket_1x04_P2.54mm_Vertical
- J3: footprint Connector_PinHeader_1.00mm:PinHeader_1x04_P1.00mm_Vertical -> Connector_PinHeader_2.54mm:PinHeader_1x04_P2.54mm_Vertical
- moved F1 5.72 mm to (232.4, 150.3)
- moved J6 5.38 mm to (168.8, 77.6), turned to 180 degrees
- moved J2 3.21 mm to (75.1, 104.7), turned to -90 degrees
- moved J10 2.92 mm to (87.3, 104.9), turned to 90 degrees
- moved Q6 2.75 mm to (245.8, 92.5), turned to 180 degrees
- moved R5 2.34 mm to (269.5, 110.8), turned to 180 degrees
- moved J1 1.70 mm to (248.5, 74.8), turned to 180 degrees
- moved D1 1.49 mm to (210.0, 142.2), turned to -90 degrees
- turned SW2 to 180 degrees
Connections:
- R1 pad 2: Net-(J7-Pin_2) -> Net-(J16-Pin_3)
- R7 pad 2: Net-(J7-Pin_3) -> Net-(J14-Pin_21)

Commit message: Can Pull
Parts:
- removed the J2 at (75.1, 104.7)
- removed the J7 at (75.7, 117.9)
- J14, J16: moved to B.Cu
- moved J14 149.9 mm to (62.8, 169.6), turned to -90 degrees
- moved J7 113.3 mm to (41.8, 130.9)
- moved J9 100.0 mm to (69.9, 186.9), turned to 90 degrees
- moved J16 91.7 mm to (62.7, 108.7), turned to -90 degrees
- moved J10 85.8 mm to (110.0, 187.7)
- moved J6 85.2 mm to (84.2, 67.6), turned to 0 degrees
- moved J12 66.6 mm to (115.0, 100.0)
- moved J2 65.4 mm to (91.8, 122.0), turned to 90 degrees
- moved F4 65.4 mm to (89.7, 80.4), turned to -90 degrees
- moved Q17 60.6 mm to (87.4, 88.9), turned to 0 degrees
- moved D4 57.0 mm to (87.2, 94.6), turned to 180 degrees
- moved J11 53.6 mm to (52.7, 97.6)
- moved R8 50.9 mm to (90.1, 98.7), turned to 0 degrees
- moved R10 49.4 mm to (93.2, 94.6), turned to 0 degrees
- moved R12 39.5 mm to (70.1, 95.8)
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
Commit message: Can Pull
Parts:
- moved J10 111.8 mm to (133.5, 78.4), turned to 180 degrees
- moved J9 94.9 mm to (135.2, 118.0), turned to 180 degrees
- moved F3 84.7 mm to (96.4, 64.4), turned to -90 degrees
- moved C8 81.6 mm to (98.0, 67.7), turned to 0 degrees
- moved J4 80.0 mm to (90.1, 65.2), turned to 90 degrees
- moved C9 78.2 mm to (98.0, 70.5), turned to 0 degrees
- moved J6 74.3 mm to (19.2, 103.6), turned to 90 degrees
- moved J14 73.6 mm to (121.3, 125.0), turned to 0 degrees
- moved R19 71.7 mm to (98.2, 76.0), turned to 0 degrees
- moved U6 70.9 mm to (91.3, 72.8), turned to 90 degrees
- moved J12 68.9 mm to (51.6, 72.8), turned to 90 degrees
- moved C10 65.6 mm to (94.7, 78.9), turned to 0 degrees
- moved R18 61.1 mm to (90.1, 79.9), turned to -90 degrees
- moved F4 60.3 mm to (32.0, 98.1), turned to 0 degrees
- moved R17 58.7 mm to (93.4, 83.9), turned to 90 degrees
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
Commit message: Can Pull
Parts:
- moved F3 17.2 mm to (104.4, 79.6), turned to 180 degrees
- moved C4 14.7 mm to (87.0, 112.7), turned to 180 degrees
- moved C8 13.9 mm to (101.1, 81.2), turned to -90 degrees
- moved C6 13.7 mm to (87.0, 110.0), turned to 180 degrees
- moved R20 13.6 mm to (105.6, 112.1), turned to 180 degrees
- moved F2 12.2 mm to (88.7, 105.3), turned to -90 degrees
- moved R15 11.9 mm to (100.5, 116.2), turned to -90 degrees
- moved R17 11.2 mm to (84.9, 76.6), turned to 0 degrees
- moved C9 10.7 mm to (98.3, 81.2), turned to -90 degrees
- moved J5 9.72 mm to (95.8, 122.1)
- moved R19 7.60 mm to (92.8, 81.4), turned to -90 degrees
- moved U4 7.03 mm to (94.5, 113.2), turned to 180 degrees
- moved J4 6.99 mm to (96.8, 67.2)
- moved R18 6.70 mm to (88.9, 73.3), turned to 180 degrees
- moved C5 6.21 mm to (100.6, 110.5), turned to 90 degrees
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
Commit message: Can Pull
Parts:
- moved J7 41.7 mm to (111.5, 146.6)
- moved R1 41.7 mm to (113.7, 141.2)
- moved R7 41.7 mm to (124.3, 141.0)
- moved J4 18.5 mm to (79.1, 72.5)
- moved U6 18.5 mm to (78.3, 79.9)
- moved C8 18.5 mm to (83.4, 86.5)
- moved C9 18.5 mm to (80.6, 86.5)
- moved R19 18.5 mm to (75.1, 86.7)
- moved R18 18.5 mm to (71.2, 78.6)
- moved C10 18.5 mm to (72.2, 83.2)
- moved F3 18.5 mm to (86.7, 84.9)
- moved R17 18.5 mm to (67.2, 81.9)
- moved J2 8.51 mm to (68.4, 102.7)
- moved C5 5.01 mm to (103.0, 114.9)
- moved C6 5.01 mm to (89.4, 114.4)
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